Commit message: updated URDF and controllers

File: ur5e_hande/urdf/ur5e_hande.urdf (robot description, URDF)
Before this commit: robot ur5e_hande, 15 links, 14 joints
Links:
- added link world
Joints:
- added joint world_joint: type fixed, parent world, child base_link, origin xyz=0.0 0.0 0.0 rpy=0.0 0.0 0.0

File: ur5e_hande/urdf/ur5e_hande.xacro (robot description, xacro)
@@ -11,3 +11,9 @@
         <origin xyz="0.0 0.0 0.0" rpy="0 1.57 0" />
     </joint> -->
+    <link name="world" />
+    <joint name="world_joint" type="fixed">
+        <parent link="world" />
+        <child link = "base_link" />
+        <origin xyz="0.0 0.0 0.0" rpy="0.0 0.0 0.0" />
+    </joint>
 </robot>
