Commit message: updated joint name

File: ur5e_hande/urdf/ur5e_hande_orig.urdf (robot description, URDF)
Before this commit: robot ur5e_hande, 16 links, 15 joints
Joints:
- removed joint finger_joint
- added joint hande_left_finger_joint: type prismatic, parent hand_e_link, child hande_left_finger, origin xyz=0 0 0.099 rpy=0 0 0, axis -1 0 0, limit lower=0 upper=0.025 effort=130 velocity=0.15
- joint hande_right_finger_joint: mimic joint=finger_joint multiplier=1 offset=0 -> joint=hande_left_finger_joint multiplier=1 offset=0
